Commit message: Add files via upload

File: Project2/workspace/catkin_ws/src/my_robot/urdf/my_robot.xacro (robot description, xacro)
@@ -149,5 +149,5 @@
   </link>
   <joint type="continuous" name="left_wheel_hinge">
-    <origin xyz="0 0.55 0" rpy="0 0 0"/>
+    <origin xyz="0 0.53 0" rpy="0 0 0"/>
     <child link="left_wheel"/>
     <parent link="chassis"/>
@@ -157,5 +157,5 @@
   </joint>
   <joint type="continuous" name="right_wheel_hinge">
-    <origin xyz="0 -0.55 0" rpy="0 0 0"/>
+    <origin xyz="0 -0.53 0" rpy="0 0 0"/>
     <child link="right_wheel"/>
     <parent link="chassis"/>
